File: KiCAD/vpc-32-v3/vpc-32-v3.sch (KiCad schematic (older format))
At the start: 67 parts, among them J1 BARREL_JACK, J2 PIC32_ICSP, J3 keyboard, J4 SD_Card, J5 VGA out, J6 PIC12_ICSP, J7 AUDIO OUTPUT, J8 RJ12, Q1 2N3904, Q2 2N3906, SW1 SPDT, SW2 ~RESET, U1 LM7805, U2 PIC12F1572, U3 LM1117-3.3, U4 PIC32MX170F256B, U5 23LC512, Y1 10Mhz

Commit message: modification à keyboard.c et edit.c ans vm.h remplacé les '#define' des opcodes par une énumération. Retiré vpcBasic du projet. Modification à la schématique pour ajouter l'ampli audio LM386.
Parts:
- removed C10: 10nF, symbol C
- removed J7: AUDIO OUTPUT, symbol CONN_COAXIAL
- removed R15: 680, symbol R
- added C11, C16: 10µF, symbol CP
- added C18: 47nF, symbol C
- added C19: 220µF, symbol CP
- added LS1: 8 ohm, symbol Speaker
- added R18: 10, symbol R
- added RV1: 10K, symbol POT
- added U5: LM386, symbol LM386
- gave numbers to parts that had none: 2
- renumbered C9 to C10, C11 to C12, C12 to C13, C13 to C14, C14 to C15, C15 to C17, C16 to C20, C17 to C21, J8 to J7, R8 to R10, R9 to R11, R10 to R12, R11 to R13, R12 to R14, R13 to R15, R14 to R16, R16 to R19, R17 to R20, R18 to R21, R19 to R22, R20 to R23, R21 to R24, R6 to R8, R7 to R9, U5 to U6
Connections:
- net +5v: now also U5.6 (V+)
- net GND: now also C16.2, C18.2, LS1.2, RV1.3, U5.2 (-), U5.4 (Gnd)
- net at R16.1: now also C11.1
- new net: RV1.2, U5.3 (+)
- new net: C19.1, R18.1, U5.5
- new net: C16.1, U5.7
- new net: C18.1, R18.2
- new net: C19.2, LS1.1
- new net: C11.2, RV1.1
Other:
- moved on the sheet: R16
